Commit message: Lab2 rodear imcompleto

File: autlab2/urdf/aubot.urdf (robot description, URDF)
Before this commit: robot aubot, 7 links, 6 joints
Joints:
- joint top_sensor_joint: origin xyz=0 0 0.0425 rpy=0 0 0 -> xyz=0 0 0.07 rpy=0 0 0

Commit message: LiDAR Arreglado

File: autlab2/urdf/aubot.urdf (robot description, URDF)
Before this commit: robot aubot, 7 links, 6 joints
Joints:
- joint top_sensor_joint: origin xyz=0 0 0.07 rpy=0 0 0 -> xyz=0 0 0.08 rpy=0 0 0
